File: hw/usb_if.sch (EAGLE design)
At the start: 5 parts, among them X1 USB-A-H

Commit message: Revert "Added ferrite bead"
This reverts commit 0db771cb7db5912f6d11f821d302d115756e7d79.
Parts:
- removed FB1: BLM15HB121SN1, inductors:BLM15HB121SN1
Connections:
- removed net N$8: FB1.1, X1.D-
- net N$6: now also X1.D-; no longer FB1.2
Changed lines of the file:
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@@
 <part name="LED1" library="WS2812B" deviceset="WS2812B" device="3535"/>
 <part name="GND6" library="supply1" library_urn="urn:adsk.eagle:library:371" deviceset="GND" device=""/>
-<part name="FB1" library="inductors" library_urn="urn:adsk.eagle:library:243" deviceset="BLM15H" device="" package3d_urn="urn:adsk.eagle:package:15132/1" technology="B121SN1"/>
 </parts>
 <sheets>
@@
 </instance>
 <instance part="R4" gate="G$1" x="101.6" y="55.88" smashed="yes" rot="R90">
-<attribute name="TAG" x="99.06" y="58.42" size="1.778" layer="96" rot="R180"/>
+<attribute name="TAG" x="104.14" y="55.88" size="1.778" layer="96"/>
 </instance>
 <instance part="P+2" gate="1" x="2.54" y="68.58" smashed="yes">
@@
 <instance part="GND6" gate="1" x="86.36" y="10.16" smashed="yes">
 <attribute name="VALUE" x="83.82" y="7.62" size="1.778" layer="96"/>
-</instance>
-<instance part="FB1" gate="G$1" x="111.76" y="55.88" smashed="yes" rot="R90">
-<attribute name="NAME" x="110.49" y="59.5884" size="1.778" layer="95" rot="R180"/>
 </instance>
 </instances>
@@
 <net name="N$6" class="0">
 <segment>
+<wire x1="111.76" y1="63.5" x2="111.76" y2="50.8" width="0.1524" layer="91"/>
 <wire x1="134.62" y1="58.42" x2="134.62" y2="63.5" width="0.1524" layer="91"/>
 <wire x1="134.62" y1="63.5" x2="111.76" y2="63.5" width="0.1524" layer="91"/>
 <junction x="111.76" y="63.5"/>
 <wire x1="96.52" y1="63.5" x2="101.6" y2="63.5" width="0.1524" layer="91"/>
+<pinref part="X1" gate="G$1" pin="D-"/>
 <wire x1="101.6" y1="63.5" x2="111.76" y2="63.5" width="0.1524" layer="91"/>
+<wire x1="111.76" y1="50.8" x2="116.84" y2="50.8" width="0.1524" layer="91"/>
 <wire x1="101.6" y1="60.96" x2="101.6" y2="63.5" width="0.1524" layer="91"/>
 <junction x="101.6" y="63.5"/>
-<wire x1="111.76" y1="63.5" x2="111.76" y2="60.96" width="0.1524" layer="91"/>
-<pinref part="FB1" gate="G$1" pin="2"/>
 </segment>
 </net>
@@
 <wire x1="50.8" y1="53.34" x2="50.8" y2="63.5" width="0.1524" layer="91"/>
 <wire x1="86.36" y1="63.5" x2="50.8" y2="63.5" width="0.1524" layer="91"/>
-</segment>
-</net>
-<net name="N$8" class="0">
-<segment>
-<pinref part="X1" gate="G$1" pin="D-"/>
-<wire x1="111.76" y1="50.8" x2="116.84" y2="50.8" width="0.1524" layer="91"/>
-<pinref part="FB1" gate="G$1" pin="1"/>
-<junction x="111.76" y="50.8"/>
 </segment>
 </net>
@@
 will not be understood (or retained) with this version.
 </note>
-<note version="8.3" severity="warning">
-Since Version 8.3, EAGLE supports the association of 3D packages
-with devices in libraries, schematics, and board files. Those 3D
-packages will not be understood (or retained) with this version.
-</note>
 <note version="8.4" severity="warning">
